Commit message: Change the urdf intial positions and only deploy stance pose after spawning

File: resources/mini_cheetah/mini_cheetah.urdf (robot description, URDF)
Before this commit: robot mini_cheetah, 17 links, 16 joints
Joints:
- joint abduct_fl_to_thigh_fl_j: origin xyz=0.0 0.062 0.00 rpy=0.0 0.6 0.0 -> xyz=0.0 0.062 0.00 rpy=0.0 0.0 0.0
- joint abduct_fr_to_thigh_fr_j: origin xyz=0.0 -0.062 0.00 rpy=0.0 0.6 0.0 -> xyz=0.0 -0.062 0.00 rpy=0.0 0.0 0.0
- joint abduct_hl_to_thigh_hl_j: origin xyz=0.0 0.062 0.00 rpy=0.0 0.6 0.0 -> xyz=0.0 0.062 0.00 rpy=0.0 0.0 0.0
- joint abduct_hr_to_thigh_hr_j: origin xyz=0.0 -0.062 0.00 rpy=0.0 0.6 0.0 -> xyz=0.0 -0.062 0.00 rpy=0.0 0.0 0.0
- joint thigh_fl_to_knee_fl_j: origin xyz=0.0 0.0 -0.209 rpy=0.0 -1.5 0.0 -> xyz=0.0 0.0 -0.209 rpy=0.0 0.0 0.0
- joint thigh_fr_to_knee_fr_j: origin xyz=0.0 0.0 -0.209 rpy=0.0 -1.5 0.0 -> xyz=0.0 0.0 -0.209 rpy=0.0 0.0 0.0
- joint thigh_hl_to_knee_hl_j: origin xyz=0.0 0.0 -0.209 rpy=0.0 -1.5 0.0 -> xyz=0.0 0.0 -0.209 rpy=0.0 0.0 0.0
- joint thigh_hr_to_knee_hr_j: origin xyz=0.0 0.0 -0.209 rpy=0.0 -1.5 0.0 -> xyz=0.0 0.0 -0.209 rpy=0.0 0.0 0.0

File: resources/mini_cheetah/mini_cheetah_skeleton.urdf (robot description, URDF)
Before this commit: robot mini_cheetah, 17 links, 16 joints
Joints:
- joint abduct_fl_to_thigh_fl_j: origin xyz=0.0 0.062 0.00 rpy=0.0 0.6 0.0 -> xyz=0.0 0.062 0.00 rpy=0.0 0.0 0.0
- joint abduct_fr_to_thigh_fr_j: origin xyz=0.0 -0.062 0.00 rpy=0.0 0.6 0.0 -> xyz=0.0 -0.062 0.00 rpy=0.0 0.0 0.0
- joint abduct_hl_to_thigh_hl_j: origin xyz=0.0 0.062 0.00 rpy=0.0 0.6 0.0 -> xyz=0.0 0.062 0.00 rpy=0.0 0.0 0.0
- joint abduct_hr_to_thigh_hr_j: origin xyz=0.0 -0.062 0.00 rpy=0.0 0.6 0.0 -> xyz=0.0 -0.062 0.00 rpy=0.0 0.0 0.0
- joint thigh_fl_to_knee_fl_j: origin xyz=0.0 0.0 -0.209 rpy=0.0 -1.5 0.0 -> xyz=0.0 0.0 -0.209 rpy=0.0 0.0 0.0
- joint thigh_fr_to_knee_fr_j: origin xyz=0.0 0.0 -0.209 rpy=0.0 -1.5 0.0 -> xyz=0.0 0.0 -0.209 rpy=0.0 0.0 0.0
- joint thigh_hl_to_knee_hl_j: origin xyz=0.0 0.0 -0.209 rpy=0.0 -1.5 0.0 -> xyz=0.0 0.0 -0.209 rpy=0.0 0.0 0.0
- joint thigh_hr_to_knee_hr_j: origin xyz=0.0 0.0 -0.209 rpy=0.0 -1.5 0.0 -> xyz=0.0 0.0 -0.209 rpy=0.0 0.0 0.0
