Commit message: Changed to skeleton urdf for faster simulation during testing

File: resources/mini_cheetah/mini_cheetah_skeleton.urdf (robot description, URDF)
Before this commit: robot mini_cheetah, 17 links, 16 joints
Links:
- link abduct_fl: geometry collision mesh filename=/home/liew/my_projects/simulation_quadruped/resources/mini_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; visual mesh filename=/home/liew/my_projects/simulation_quadruped/resources/mini_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
- link abduct_fr: geometry collision mesh filename=/home/liew/my_projects/simulation_quadruped/resources/mini_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; visual mesh filename=/home/liew/my_projects/simulation_quadruped/resources/mini_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
- link abduct_hl: geometry collision mesh filename=/home/liew/my_projects/simulation_quadruped/resources/mini_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; visual mesh filename=/home/liew/my_projects/simulation_quadruped/resources/mini_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
- link abduct_hr: geometry collision mesh filename=/home/liew/my_projects/simulation_quadruped/resources/mini_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; visual mesh filename=/home/liew/my_projects/simulation_quadruped/resources/mini_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
- link body: geometry collision mesh filename=/home/liew/my_projects/simulation_quadruped/resources/mini_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; visual mesh filename=/home/liew/my_projects/simulation_quadruped/resources/mini_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
- link shank_fl: geometry collision mesh filename=/home/liew/my_projects/simulation_quadruped/resources/mini_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; visual mesh filename=/home/liew/my_projects/simulation_quadruped/resources/mini_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
- link shank_fr: geometry collision mesh filename=/home/liew/my_projects/simulation_quadruped/resources/mini_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; visual mesh filename=/home/liew/my_projects/simulation_quadruped/resources/mini_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
- link shank_hl: geometry collision mesh filename=/home/liew/my_projects/simulation_quadruped/resources/mini_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; visual mesh filename=/home/liew/my_projects/simulation_quadruped/resources/mini_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
- link shank_hr: geometry collision mesh filename=/home/liew/my_projects/simulation_quadruped/resources/mini_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; visual mesh filename=/home/liew/my_projects/simulation_quadruped/resources/mini_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
- link thigh_fl: geometry collision mesh filename=/home/liew/my_projects/simulation_quadruped/resources/mini_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; visual mesh filename=/home/liew/my_projects/simulation_quadruped/resources/mini_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
- link thigh_fr: geometry collision mesh filename=/home/liew/my_projects/simulation_quadruped/resources/mini_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; visual mesh filename=/home/liew/my_projects/simulation_quadruped/resources/mini_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
- link thigh_hl: geometry collision mesh filename=/home/liew/my_projects/simulation_quadruped/resources/mini_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; visual mesh filename=/home/liew/my_projects/simulation_quadruped/resources/mini_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
- link thigh_hr: geometry collision mesh filename=/home/liew/my_projects/simulation_quadruped/resources/mini_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; visual mesh filename=/home/liew/my_projects/simulation_quadruped/resources/mini_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
