Commit message: Added cmake files to find quadruped control library and enlarge ground size

File: resources/ground.urdf (robot description, URDF)
Before this commit: robot ground_skeleton, 2 links, 1 joints
Links:
- link ground_link: geometry collision box size=2.0 0.05 2.0; visual box size=10.0 0.05 10.0

Commit message: Implemented PD control and fixed urdf (forgot to modify collision)

File: resources/ground.urdf (robot description, URDF)
Before this commit: robot ground_skeleton, 2 links, 1 joints
Links:
- link ground_link: geometry collision box size=10.0 0.05 10.0; visual box size=10.0 0.05 10.0
